Commit message: imu_description : add generation of urdf file

File: romea_imu_description/urdf/imu.xacro (robot description, xacro)
@@ -2,10 +2,9 @@
 <robot name="imu"
   xmlns:xacro="http://www.ros.org/wiki/xacro">
-  <xacro:macro name="imu_sensor" params="xyz rpy parent_link rate type model name">
+  <xacro:macro name="imu_sensor" params="xyz rpy parent_link rate type model name prefix">
     <xacro:property name="conf" value="$(find romea_imu_description)/config/${type}_${model}.yaml" />
     <xacro:property name="props" value="${load_yaml(conf)}"/>
     <xacro:property name="link_name" value="${prefix}${name}_link"/>
     <xacro:property name="joint_name" value="${prefix}${name}_joint"/>
-    <xacro:property name="controller_name" value="${prefix}${name}_controller"/>
     <xacro:property name="parent_link_name" value="${prefix}${parent_link}"/>
     <xacro:property name="data_topic" value="${name}/data"/>
@@ -15,7 +14,4 @@
     <xacro:property name="ang_drift_std" value="${props['angular_speed_bias_stability_std']}"/>
     <xacro:property name="heading_std" value="${props['heading_std']}"/>
-    <gazebo reference="${link_name}">
-      <material>Gazebo/Orange</material>
-    </gazebo>
     <link name="${link_name}">
       <visual>
@@ -32,22 +28,58 @@
     </joint>
     <gazebo reference="${link_name}">
-      <gravity>true</gravity>
-      <sensor name='imu_sensor' type='imu'>
-        <always_on>1</always_on>
-        <update_rate>1000</update_rate>
-        <visualize>1</visualize>
-        <topic>__default_topic__</topic>
-        <plugin name="${controller_name}" filename="libgazebo_ros_romea_imu.so">
-          <update_rate>${rate}</update_rate>
-          <body_name>${parent_link}</body_name>
-          <topic_name>${name}/data</topic_name>
-          <link_name>${link_name}</link_name>
-          <accel_std>${acc_noise_std}</accel_std>
-          <rate_std>${ang_noise_std}</rate_std>
-          <angle_std>${heading_std}</angle_std>
-          <imu_name>${prefix}${name}</imu_name>
-        </plugin>
-        <pose>0 0 0 0 0 0</pose>
-      </sensor>
+        <material>Gazebo/Orange</material>
+        <sensor name="${name}" type="imu">
+            <always_on>true</always_on>
+            <update_rate>100</update_rate>
+            <imu>
+              <angular_velocity>
+                <x>
+                  <noise type="gaussian">
+                    <mean>0.0</mean>
+                    <stddev>${ang_noise_std}</stddev>
+                  </noise>
+                </x>
+                <y>
+                  <noise type="gaussian">
+                    <mean>0.0</mean>
+                    <stddev>${ang_noise_std}</stddev>
+                  </noise>
+                </y>
+                <z>
+                  <noise type="gaussian">
+                    <mean>0.0</mean>
+                    <stddev>${ang_noise_std}</stddev>
+                  </noise>
+                </z>
+              </angular_velocity>
+              <linear_acceleration>
+                <x>
+                  <noise type="gaussian">
+                    <mean>0.0</mean>
+                    <stddev>${acc_noise_std}</stddev>
+                  </noise>
+                </x>
+                <y>
+                  <noise type="gaussian">
+                    <mean>0.0</mean>
+                    <stddev>${acc_noise_std}</stddev>
+                  </noise>
+                </y>
+                <z>
+                  <noise type="gaussian">
+                    <mean>0.0</mean>
+                    <stddev>${acc_noise_std}</stddev>
+                  </noise>
+                </z>
+              </linear_acceleration>
+            </imu>
+            <plugin name="${name}" filename="libgazebo_ros_imu_sensor.so">
+                <ros>
+                    <namespace>${prefix}${name}</namespace>
+                    <remapping>~/out:=${name}/data</remapping>
+                </ros>
+                <initial_orientation_as_reference>false</initial_orientation_as_reference>
+            </plugin>
+        </sensor>
     </gazebo>
   </xacro:macro>

Commit message: imu_description:  add geometry description  + mesh description

File: romea_imu_description/urdf/imu.xacro (robot description, xacro)
@@ -2,22 +2,55 @@
 <robot name="imu"
   xmlns:xacro="http://www.ros.org/wiki/xacro">
-  <xacro:macro name="imu_sensor" params="xyz rpy parent_link rate type model name prefix">
-    <xacro:property name="conf" value="$(find romea_imu_description)/config/${type}_${model}.yaml" />
-    <xacro:property name="props" value="${load_yaml(conf)}"/>
+  <xacro:macro name="imu_sensor" params="xyz rpy parent_link rate type model name prefix mesh_visual">
+    <xacro:property name="specifications_file" value="$(find romea_imu_description)/config/${type}_${model}_specifications.yaml" />
+    <xacro:property name="geometry_file" value="$(find romea_imu_description)/config/${type}_${model}_geometry.yaml" />
+    <xacro:property name="specifications" value="${load_yaml(specifications_file)}"/>
+    <xacro:property name="geometry" value="${load_yaml(geometry_file)}"/>
     <xacro:property name="link_name" value="${prefix}${name}_link"/>
     <xacro:property name="joint_name" value="${prefix}${name}_joint"/>
     <xacro:property name="parent_link_name" value="${prefix}${parent_link}"/>
     <xacro:property name="data_topic" value="${name}/data"/>
-    <xacro:property name="acc_noise_std" value="${1.57*props['acceleration_noise_density']*sqrt(rate)}"/>
-    <xacro:property name="acc_drift_std" value="${props['acceleration_bias_stability_std']}"/>
-    <xacro:property name="ang_noise_std" value="${1.57*props['angular_speed_noise_density']*sqrt(rate)}"/>
-    <xacro:property name="ang_drift_std" value="${props['angular_speed_bias_stability_std']}"/>
-    <xacro:property name="heading_std" value="${props['heading_std']}"/>
+    <xacro:property name="acc_noise_std" value="${1.57*specifications['acceleration_noise_density']*sqrt(rate)}"/>
+    <xacro:property name="acc_drift_std" value="${specifications['acceleration_bias_stability_std']}"/>
+    <xacro:property name="ang_noise_std" value="${1.57*specifications['angular_speed_noise_density']*sqrt(rate)}"/>
+    <xacro:property name="ang_drift_std" value="${specifications['angular_speed_bias_stability_std']}"/>
+    <xacro:property name="heading_std" value="${specifications['heading_std']}"/>
+    <xacro:property name="mass" value="${geometry['mass']}"/>
+    <xacro:property name="aabb_length" value="${geometry['aabb']['length']}"/>
+    <xacro:property name="aabb_width" value="${geometry['aabb']['width']}"/>
+    <xacro:property name="aabb_height" value="${geometry['aabb']['height']}"/>
+    <xacro:property name="aabb_center" value="${geometry['aabb']['center']}"/>
+    <xacro:property name="mesh_xyz" value="${geometry['mesh']['xyz']}"/>
+    <xacro:property name="mesh_rpy" value="${geometry['mesh']['rpy']}"/>
+    <xacro:property name="mesh_scale" value="${geometry['mesh']['scale']}"/>
+    <xacro:property name="mesh_filename" value="${geometry['mesh']['filename']}"/>
     <link name="${link_name}">
-      <visual>
-        <geometry>
-          <box size="0.03 0.05 0.02"/>
-        </geometry>
-      </visual>
+       <inertial>
+         <mass value="${mass}" />
+         <origin xyz="${aabb_center[0]} ${aabb_center[1]} ${aabb_center[2]}" />
+         <inertia ixx="${0.0833333 * mass * (aabb_width*aabb_width + aabb_height*aabb_height)}" ixy="0.0" ixz="0.0"
+           iyy="${0.0833333 * mass * (aabb_height*aabb_height + aabb_length*aabb_length)}" iyz="0.0"
+           izz="${0.0833333 * mass * (aabb_length*aabb_length + aabb_width*aabb_width)}" />
+       </inertial>
+       <visual>
+         <xacro:if value="${mesh_visual == True}">
+            <origin xyz="${mesh_xyz[0]} ${mesh_xyz[1]} ${mesh_xyz[2]}" rpy="${mesh_rpy[0]} ${mesh_rpy[1]} ${mesh_rpy[2]}" />
+            <geometry>
+              <mesh filename="${mesh_filename}" scale="${mesh_scale[0]} ${mesh_scale[1]} ${mesh_scale[2]}"/>
+            </geometry>
+         </xacro:if>
+         <xacro:if value="${mesh_visual == False}">
+            <origin xyz="${aabb_center[0]} ${aabb_center[1]} ${aabb_center[2]}" rpy="0 0 0" />
+            <geometry>
+              <box size="${aabb_length} ${aabb_width} ${aabb_height}" />
+            </geometry>
+         </xacro:if>
+       </visual>
+       <collision>
+         <origin xyz="${aabb_center[0]} ${aabb_center[1]} ${aabb_center[2]}" rpy="0 0 0" />
+         <geometry>
+           <box size="${aabb_length} ${aabb_width} ${aabb_height}" />
+         </geometry>
+       </collision>
     </link>
     <joint name="${joint_name}" type="fixed">

Commit message: description : mesh visual is available if mesh description is given in geometry yaml

File: romea_imu_description/urdf/imu.xacro (robot description, xacro)
@@ -21,8 +21,10 @@
     <xacro:property name="aabb_height" value="${geometry['aabb']['height']}"/>
     <xacro:property name="aabb_center" value="${geometry['aabb']['center']}"/>
-    <xacro:property name="mesh_xyz" value="${geometry['mesh']['xyz']}"/>
-    <xacro:property name="mesh_rpy" value="${geometry['mesh']['rpy']}"/>
-    <xacro:property name="mesh_scale" value="${geometry['mesh']['scale']}"/>
-    <xacro:property name="mesh_filename" value="${geometry['mesh']['filename']}"/>
+    <xacro:if value="${mesh_visual == True and 'mesh' in geometry}">
+      <xacro:property name="mesh_xyz" value="${geometry['mesh']['xyz']}"/>
+      <xacro:property name="mesh_rpy" value="${geometry['mesh']['rpy']}"/>
+      <xacro:property name="mesh_scale" value="${geometry['mesh']['scale']}"/>
+      <xacro:property name="mesh_filename" value="${geometry['mesh']['filename']}"/>
+    </xacro:if>
     <link name="${link_name}">
        <inertial>
@@ -34,5 +36,5 @@
        </inertial>
        <visual>
-         <xacro:if value="${mesh_visual == True}">
+         <xacro:if value="${mesh_visual == True and 'mesh' in geometry}">
             <origin xyz="${mesh_xyz[0]} ${mesh_xyz[1]} ${mesh_xyz[2]}" rpy="${mesh_rpy[0]} ${mesh_rpy[1]} ${mesh_rpy[2]}" />
             <geometry>
@@ -40,5 +42,5 @@
             </geometry>
          </xacro:if>
-         <xacro:if value="${mesh_visual == False}">
+         <xacro:if value="${mesh_visual == False or 'mesh' not in geometry}">
             <origin xyz="${aabb_center[0]} ${aabb_center[1]} ${aabb_center[2]}" rpy="0 0 0" />
             <geometry>

Commit message: update to take into account additionnal ros_namespace in description

File: romea_imu_description/urdf/imu.xacro (robot description, xacro)
@@ -2,119 +2,135 @@
 <robot name="imu"
   xmlns:xacro="http://www.ros.org/wiki/xacro">
-  <xacro:macro name="imu_sensor" params="xyz rpy parent_link rate type model name prefix mesh_visual">
-    <xacro:property name="specifications_file" value="$(find romea_imu_description)/config/${type}_${model}_specifications.yaml" />
-    <xacro:property name="geometry_file" value="$(find romea_imu_description)/config/${type}_${model}_geometry.yaml" />
-    <xacro:property name="specifications" value="${load_yaml(specifications_file)}"/>
-    <xacro:property name="geometry" value="${load_yaml(geometry_file)}"/>
-    <xacro:property name="link_name" value="${prefix}${name}_link"/>
-    <xacro:property name="joint_name" value="${prefix}${name}_joint"/>
-    <xacro:property name="parent_link_name" value="${prefix}${parent_link}"/>
-    <xacro:property name="data_topic" value="${name}/data"/>
-    <xacro:property name="acc_noise_std" value="${1.57*specifications['acceleration_noise_density']*sqrt(rate)}"/>
-    <xacro:property name="acc_drift_std" value="${specifications['acceleration_bias_stability_std']}"/>
-    <xacro:property name="ang_noise_std" value="${1.57*specifications['angular_speed_noise_density']*sqrt(rate)}"/>
-    <xacro:property name="ang_drift_std" value="${specifications['angular_speed_bias_stability_std']}"/>
-    <xacro:property name="heading_std" value="${specifications['heading_std']}"/>
-    <xacro:property name="mass" value="${geometry['mass']}"/>
-    <xacro:property name="aabb_length" value="${geometry['aabb']['length']}"/>
-    <xacro:property name="aabb_width" value="${geometry['aabb']['width']}"/>
-    <xacro:property name="aabb_height" value="${geometry['aabb']['height']}"/>
-    <xacro:property name="aabb_center" value="${geometry['aabb']['center']}"/>
+  <xacro:macro name="imu_sensor"
+    params="xyz rpy parent_link rate type model name prefix mesh_visual ros_namespace">
+    <xacro:property name="specifications_file"
+      value="$(find romea_imu_description)/config/${type}_${model}_specifications.yaml" />
+    <xacro:property name="geometry_file"
+      value="$(find romea_imu_description)/config/${type}_${model}_geometry.yaml" />
+    <xacro:property name="specifications"
+      value="${load_yaml(specifications_file)}" />
+    <xacro:property name="geometry"
+      value="${load_yaml(geometry_file)}" />
+    <xacro:property name="link_name"
+      value="${prefix}${name}_link" />
+    <xacro:property name="joint_name"
+      value="${prefix}${name}_joint" />
+    <xacro:property name="parent_link_name"
+      value="${prefix}${parent_link}" />
+    <xacro:property name="data_topic"
+      value="${name}/data" />
+    <xacro:property name="acc_noise_std"
+      value="${1.57*specifications['acceleration_noise_density']*sqrt(rate)}" />
+    <xacro:property name="acc_drift_std"
+      value="${specifications['acceleration_bias_stability_std']}" />
+    <xacro:property name="ang_noise_std"
+      value="${1.57*specifications['angular_speed_noise_density']*sqrt(rate)}" />
+    <xacro:property name="ang_drift_std"
+      value="${specifications['angular_speed_bias_stability_std']}" />
+    <xacro:property name="heading_std" value="${specifications['heading_std']}" />
+    <xacro:property name="mass" value="${geometry['mass']}" />
+    <xacro:property name="aabb_length" value="${geometry['aabb']['length']}" />
+    <xacro:property name="aabb_width" value="${geometry['aabb']['width']}" />
+    <xacro:property name="aabb_height" value="${geometry['aabb']['height']}" />
+    <xacro:property name="aabb_center" value="${geometry['aabb']['center']}" />
     <xacro:if value="${mesh_visual == True and 'mesh' in geometry}">
-      <xacro:property name="mesh_xyz" value="${geometry['mesh']['xyz']}"/>
-      <xacro:property name="mesh_rpy" value="${geometry['mesh']['rpy']}"/>
-      <xacro:property name="mesh_scale" value="${geometry['mesh']['scale']}"/>
-      <xacro:property name="mesh_filename" value="${geometry['mesh']['filename']}"/>
+      <xacro:property name="mesh_xyz" value="${geometry['mesh']['xyz']}" />
+      <xacro:property name="mesh_rpy" value="${geometry['mesh']['rpy']}" />
+      <xacro:property name="mesh_scale" value="${geometry['mesh']['scale']}" />
+      <xacro:property name="mesh_filename" value="${geometry['mesh']['filename']}" />
     </xacro:if>
     <link name="${link_name}">
-       <inertial>
-         <mass value="${mass}" />
-         <origin xyz="${aabb_center[0]} ${aabb_center[1]} ${aabb_center[2]}" />
-         <inertia ixx="${0.0833333 * mass * (aabb_width*aabb_width + aabb_height*aabb_height)}" ixy="0.0" ixz="0.0"
-           iyy="${0.0833333 * mass * (aabb_height*aabb_height + aabb_length*aabb_length)}" iyz="0.0"
-           izz="${0.0833333 * mass * (aabb_length*aabb_length + aabb_width*aabb_width)}" />
-       </inertial>
-       <visual>
-         <xacro:if value="${mesh_visual == True and 'mesh' in geometry}">
-            <origin xyz="${mesh_xyz[0]} ${mesh_xyz[1]} ${mesh_xyz[2]}" rpy="${mesh_rpy[0]} ${mesh_rpy[1]} ${mesh_rpy[2]}" />
-            <geometry>
-              <mesh filename="${mesh_filename}" scale="${mesh_scale[0]} ${mesh_scale[1]} ${mesh_scale[2]}"/>
-            </geometry>
-         </xacro:if>
-         <xacro:if value="${mesh_visual == False or 'mesh' not in geometry}">
-            <origin xyz="${aabb_center[0]} ${aabb_center[1]} ${aabb_center[2]}" rpy="0 0 0" />
-            <geometry>
-              <box size="${aabb_length} ${aabb_width} ${aabb_height}" />
-            </geometry>
-         </xacro:if>
-       </visual>
-       <collision>
-         <origin xyz="${aabb_center[0]} ${aabb_center[1]} ${aabb_center[2]}" rpy="0 0 0" />
-         <geometry>
-           <box size="${aabb_length} ${aabb_width} ${aabb_height}" />
-         </geometry>
-       </collision>
+      <inertial>
+        <mass value="${mass}" />
+        <origin xyz="${aabb_center[0]} ${aabb_center[1]} ${aabb_center[2]}" />
+        <inertia ixx="${0.0833333 * mass * (aabb_width*aabb_width + aabb_height*aabb_height)}"
+          ixy="0.0" ixz="0.0"
+          iyy="${0.0833333 * mass * (aabb_height*aabb_height + aabb_length*aabb_length)}" iyz="0.0"
+          izz="${0.0833333 * mass * (aabb_length*aabb_length + aabb_width*aabb_width)}" />
+      </inertial>
+      <visual>
+        <xacro:if value="${mesh_visual == True and 'mesh' in geometry}">
+          <origin xyz="${mesh_xyz[0]} ${mesh_xyz[1]} ${mesh_xyz[2]}"
+            rpy="${mesh_rpy[0]} ${mesh_rpy[1]} ${mesh_rpy[2]}" />
+          <geometry>
+            <mesh filename="${mesh_filename}"
+              scale="${mesh_scale[0]} ${mesh_scale[1]} ${mesh_scale[2]}" />
+          </geometry>
+        </xacro:if>
+        <xacro:if value="${mesh_visual == False or 'mesh' not in geometry}">
+          <origin xyz="${aabb_center[0]} ${aabb_center[1]} ${aabb_center[2]}" rpy="0 0 0" />
+          <geometry>
+            <box size="${aabb_length} ${aabb_width} ${aabb_height}" />
+          </geometry>
+        </xacro:if>
+      </visual>
+      <collision>
+        <origin xyz="${aabb_center[0]} ${aabb_center[1]} ${aabb_center[2]}" rpy="0 0 0" />
+        <geometry>
+          <box size="${aabb_length} ${aabb_width} ${aabb_height}" />
+        </geometry>
+      </collision>
     </link>
     <joint name="${joint_name}" type="fixed">
       <axis xyz="0 0 1" />
-      <origin xyz="${xyz}" rpy="${rpy}"/>
-      <parent link="${parent_link_name}"/>
-      <child link="${link_name}"/>
+      <origin xyz="${xyz}" rpy="${rpy}" />
+      <parent link="${parent_link_name}" />
+      <child link="${link_name}" />
     </joint>
     <gazebo reference="${link_name}">
-        <material>Gazebo/Orange</material>
-        <sensor name="${name}" type="imu">
-            <always_on>true</always_on>
-            <update_rate>100</update_rate>
-            <imu>
-              <angular_velocity>
-                <x>
-                  <noise type="gaussian">
-                    <mean>0.0</mean>
-                    <stddev>${ang_noise_std}</stddev>
-                  </noise>
-                </x>
-                <y>
-                  <noise type="gaussian">
-                    <mean>0.0</mean>
-                    <stddev>${ang_noise_std}</stddev>
-                  </noise>
-                </y>
-                <z>
-                  <noise type="gaussian">
-                    <mean>0.0</mean>
-                    <stddev>${ang_noise_std}</stddev>
-                  </noise>
-                </z>
-              </angular_velocity>
-              <linear_acceleration>
-                <x>
-                  <noise type="gaussian">
-                    <mean>0.0</mean>
-                    <stddev>${acc_noise_std}</stddev>
-                  </noise>
-                </x>
-                <y>
-                  <noise type="gaussian">
-                    <mean>0.0</mean>
-                    <stddev>${acc_noise_std}</stddev>
-                  </noise>
-                </y>
-                <z>
-                  <noise type="gaussian">
-                    <mean>0.0</mean>
-                    <stddev>${acc_noise_std}</stddev>
-                  </noise>
-                </z>
-              </linear_acceleration>
-            </imu>
-            <plugin name="${name}" filename="libgazebo_ros_imu_sensor.so">
-                <ros>
-                    <!-- <namespace>${prefix}${name}</namespace> --> <!-- not working -->
-                    <remapping>~/out:=${name}/data</remapping>
-                </ros>
-                <initial_orientation_as_reference>false</initial_orientation_as_reference>
-            </plugin>
-        </sensor>
+      <material>Gazebo/Orange</material>
+      <sensor name="${name}" type="imu">
+        <always_on>true</always_on>
+        <update_rate>100</update_rate>
+        <imu>
+          <angular_velocity>
+            <x>
+              <noise type="gaussian">
+                <mean>0.0</mean>
+                <stddev>${ang_noise_std}</stddev>
+              </noise>
+            </x>
+            <y>
+              <noise type="gaussian">
+                <mean>0.0</mean>
+                <stddev>${ang_noise_std}</stddev>
+              </noise>
+            </y>
+            <z>
+              <noise type="gaussian">
+                <mean>0.0</mean>
+                <stddev>${ang_noise_std}</stddev>
+              </noise>
+            </z>
+          </angular_velocity>
+          <linear_acceleration>
+            <x>
+              <noise type="gaussian">
+                <mean>0.0</mean>
+                <stddev>${acc_noise_std}</stddev>
+              </noise>
+            </x>
+            <y>
+              <noise type="gaussian">
+                <mean>0.0</mean>
+                <stddev>${acc_noise_std}</stddev>
+              </noise>
+            </y>
+            <z>
+              <noise type="gaussian">
+                <mean>0.0</mean>
+                <stddev>${acc_noise_std}</stddev>
+              </noise>
+            </z>
+          </linear_acceleration>
+        </imu>
+        <plugin name="driver" filename="libgazebo_ros_imu_sensor.so">
+          <ros>
+            <namespace>${ros_namespace}</namespace>
+            <remapping>~/out:=data</remapping>
+          </ros>
+          <initial_orientation_as_reference>false</initial_orientation_as_reference>
+        </plugin>
+      </sensor>
     </gazebo>
   </xacro:macro>
