Commit message: take into account mode in urdf description

File: romea_imu_description/urdf/imu.xacro (robot description, xacro)
@@ -3,5 +3,5 @@
   xmlns:xacro="http://www.ros.org/wiki/xacro">
   <xacro:macro name="imu_sensor"
-    params="xyz rpy parent_link rate type model name prefix mesh_visual ros_namespace">
+    params="prefix mode name xyz rpy parent_link rate type model mesh_visual ros_namespace">
     <xacro:property name="specifications_file"
       value="$(find romea_imu_description)/config/${type}_${model}_specifications.yaml" />
@@ -78,60 +78,62 @@
       <child link="${link_name}" />
     </joint>
-    <gazebo reference="${link_name}">
-      <material>Gazebo/Orange</material>
-      <sensor name="${name}" type="imu">
-        <always_on>true</always_on>
-        <update_rate>100</update_rate>
-        <imu>
-          <angular_velocity>
-            <x>
-              <noise type="gaussian">
-                <mean>0.0</mean>
-                <stddev>${ang_noise_std}</stddev>
-              </noise>
-            </x>
-            <y>
-              <noise type="gaussian">
-                <mean>0.0</mean>
-                <stddev>${ang_noise_std}</stddev>
-              </noise>
-            </y>
-            <z>
-              <noise type="gaussian">
-                <mean>0.0</mean>
-                <stddev>${ang_noise_std}</stddev>
-              </noise>
-            </z>
-          </angular_velocity>
-          <linear_acceleration>
-            <x>
-              <noise type="gaussian">
-                <mean>0.0</mean>
-                <stddev>${acc_noise_std}</stddev>
-              </noise>
-            </x>
-            <y>
-              <noise type="gaussian">
-                <mean>0.0</mean>
-                <stddev>${acc_noise_std}</stddev>
-              </noise>
-            </y>
-            <z>
-              <noise type="gaussian">
-                <mean>0.0</mean>
-                <stddev>${acc_noise_std}</stddev>
-              </noise>
-            </z>
-          </linear_acceleration>
-        </imu>
-        <plugin name="driver" filename="libgazebo_ros_imu_sensor.so">
-          <ros>
-            <namespace>${ros_namespace}</namespace>
-            <remapping>~/out:=data</remapping>
-          </ros>
-          <initial_orientation_as_reference>false</initial_orientation_as_reference>
-        </plugin>
-      </sensor>
-    </gazebo>
+    <xacro:if value="${'simulation' in  mode}">
+      <gazebo reference="${link_name}">
+        <material>Gazebo/Orange</material>
+        <sensor name="${name}" type="imu">
+          <always_on>true</always_on>
+          <update_rate>100</update_rate>
+          <imu>
+            <angular_velocity>
+              <x>
+                <noise type="gaussian">
+                  <mean>0.0</mean>
+                  <stddev>${ang_noise_std}</stddev>
+                </noise>
+              </x>
+              <y>
+                <noise type="gaussian">
+                  <mean>0.0</mean>
+                  <stddev>${ang_noise_std}</stddev>
+                </noise>
+              </y>
+              <z>
+                <noise type="gaussian">
+                  <mean>0.0</mean>
+                  <stddev>${ang_noise_std}</stddev>
+                </noise>
+              </z>
+            </angular_velocity>
+            <linear_acceleration>
+              <x>
+                <noise type="gaussian">
+                  <mean>0.0</mean>
+                  <stddev>${acc_noise_std}</stddev>
+                </noise>
+              </x>
+              <y>
+                <noise type="gaussian">
+                  <mean>0.0</mean>
+                  <stddev>${acc_noise_std}</stddev>
+                </noise>
+              </y>
+              <z>
+                <noise type="gaussian">
+                  <mean>0.0</mean>
+                  <stddev>${acc_noise_std}</stddev>
+                </noise>
+              </z>
+            </linear_acceleration>
+          </imu>
+          <plugin name="driver" filename="libgazebo_ros_imu_sensor.so">
+            <ros>
+              <namespace>${ros_namespace}</namespace>
+              <remapping>~/out:=data</remapping>
+            </ros>
+            <initial_orientation_as_reference>false</initial_orientation_as_reference>
+          </plugin>
+        </sensor>
+      </gazebo>
+    </xacro:if>
   </xacro:macro>
 </robot>

Commit message: description : create generalized urdf xacro model
Signed-off-by: jean.laneurit <jean.laneurit@inrae.fr>

File: romea_imu_description/urdf/imu.xacro (robot description, xacro)
@@ -3,13 +3,5 @@
   xmlns:xacro="http://www.ros.org/wiki/xacro">
   <xacro:macro name="imu_sensor"
-    params="prefix mode name xyz rpy parent_link rate type model mesh_visual ros_namespace">
-    <xacro:property name="specifications_file"
-      value="$(find romea_imu_description)/config/${type}_${model}_specifications.yaml" />
-    <xacro:property name="geometry_file"
-      value="$(find romea_imu_description)/config/${type}_${model}_geometry.yaml" />
-    <xacro:property name="specifications"
-      value="${load_yaml(specifications_file)}" />
-    <xacro:property name="geometry"
-      value="${load_yaml(geometry_file)}" />
+    params="prefix mode name xyz rpy parent_link rate specifications geometry mesh_visual ros_namespace">
     <xacro:property name="link_name"
       value="${prefix}${name}_link" />

Commit message: description: add imu.simulation.xacro file
Signed-off-by: Jean Laneurit <jean.laneurit@inrae.fr>

File: romea_imu_description/urdf/imu.xacro (robot description, xacro)
@@ -12,23 +12,23 @@
     <xacro:property name="data_topic"
       value="${name}/data" />
-    <xacro:property name="acc_noise_std"
-      value="${1.57*specifications['acceleration_noise_density']*sqrt(rate)}" />
-    <xacro:property name="acc_drift_std"
-      value="${specifications['acceleration_bias_stability_std']}" />
-    <xacro:property name="ang_noise_std"
-      value="${1.57*specifications['angular_speed_noise_density']*sqrt(rate)}" />
-    <xacro:property name="ang_drift_std"
-      value="${specifications['angular_speed_bias_stability_std']}" />
-    <xacro:property name="heading_std" value="${specifications['heading_std']}" />
-    <xacro:property name="mass" value="${geometry['mass']}" />
-    <xacro:property name="aabb_length" value="${geometry['aabb']['length']}" />
-    <xacro:property name="aabb_width" value="${geometry['aabb']['width']}" />
-    <xacro:property name="aabb_height" value="${geometry['aabb']['height']}" />
-    <xacro:property name="aabb_center" value="${geometry['aabb']['center']}" />
+    <xacro:property name="mass"
+      value="${geometry['mass']}" />
+    <xacro:property name="aabb_length"
+      value="${geometry['aabb']['length']}" />
+    <xacro:property name="aabb_width"
+      value="${geometry['aabb']['width']}" />
+    <xacro:property name="aabb_height"
+      value="${geometry['aabb']['height']}" />
+    <xacro:property name="aabb_center"
+      value="${geometry['aabb']['center']}" />
     <xacro:if value="${mesh_visual == True and 'mesh' in geometry}">
-      <xacro:property name="mesh_xyz" value="${geometry['mesh']['xyz']}" />
-      <xacro:property name="mesh_rpy" value="${geometry['mesh']['rpy']}" />
-      <xacro:property name="mesh_scale" value="${geometry['mesh']['scale']}" />
-      <xacro:property name="mesh_filename" value="${geometry['mesh']['filename']}" />
+      <xacro:property name="mesh_xyz"
+        value="${geometry['mesh']['xyz']}" />
+      <xacro:property name="mesh_rpy"
+        value="${geometry['mesh']['rpy']}" />
+      <xacro:property name="mesh_scale"
+        value="${geometry['mesh']['scale']}" />
+      <xacro:property name="mesh_filename"
+        value="${geometry['mesh']['filename']}" />
     </xacro:if>
     <link name="${link_name}">
@@ -71,61 +71,13 @@
     </joint>
     <xacro:if value="${'simulation' in  mode}">
-      <gazebo reference="${link_name}">
-        <material>Gazebo/Orange</material>
-        <sensor name="${name}" type="imu">
-          <always_on>true</always_on>
-          <update_rate>100</update_rate>
-          <imu>
-            <angular_velocity>
-              <x>
-                <noise type="gaussian">
-                  <mean>0.0</mean>
-                  <stddev>${ang_noise_std}</stddev>
-                </noise>
-              </x>
-              <y>
-                <noise type="gaussian">
-                  <mean>0.0</mean>
-                  <stddev>${ang_noise_std}</stddev>
-                </noise>
-              </y>
-              <z>
-                <noise type="gaussian">
-                  <mean>0.0</mean>
-                  <stddev>${ang_noise_std}</stddev>
-                </noise>
-              </z>
-            </angular_velocity>
-            <linear_acceleration>
-              <x>
-                <noise type="gaussian">
-                  <mean>0.0</mean>
-                  <stddev>${acc_noise_std}</stddev>
-                </noise>
-              </x>
-              <y>
-                <noise type="gaussian">
-                  <mean>0.0</mean>
-                  <stddev>${acc_noise_std}</stddev>
-                </noise>
-              </y>
-              <z>
-                <noise type="gaussian">
-                  <mean>0.0</mean>
-                  <stddev>${acc_noise_std}</stddev>
-                </noise>
-              </z>
-            </linear_acceleration>
-          </imu>
-          <plugin name="driver" filename="libgazebo_ros_imu_sensor.so">
-            <ros>
-              <namespace>${ros_namespace}</namespace>
-              <remapping>~/out:=data</remapping>
-            </ros>
-            <frame_name>${link_name}</frame_name>
-            <initial_orientation_as_reference>false</initial_orientation_as_reference>
-          </plugin>
-        </sensor>
-      </gazebo>
+      <xacro:include filename="$(find romea_imu_description)/urdf/imu.simulation.xacro" />
+      <xacro:imu_sensor_simulation
+        prefix="${prefix}"
+        mode="${mode}"
+        name="${name}"
+        rate="${rate}"
+        link_name="${link_name}"
+        specifications="${specifications}"
+        ros_namespace="${ros_namespace}"/>
     </xacro:if>
   </xacro:macro>

Commit message: disable collision in URDF

File: romea_imu_description/urdf/imu.xacro (robot description, xacro)
@@ -57,10 +57,10 @@
         </xacro:if>
       </visual>
-      <collision>
+      <!-- <collision>
         <origin xyz="${aabb_center[0]} ${aabb_center[1]} ${aabb_center[2]}" rpy="0 0 0" />
         <geometry>
           <box size="${aabb_length} ${aabb_width} ${aabb_height}" />
         </geometry>
-      </collision>
+      </collision> -->
     </link>
     <joint name="${joint_name}" type="fixed">
